File: Common/STM32F446REBブレイクアウト基盤/stm32f446re_breakout_substrate/stm32f446re_breakout_substrate.kicad_sch (KiCad schematic)
At the start: 5 parts, among them J1 Conn_01x07_Socket, J2 Conn_01x04_Socket, J3 Conn_01x04_Socket, J4 Conn_01x04_Socket

Commit message: e
Parts:
- removed U1: ~, symbol MyLibrary:stm32f446re_modle
- added C1, C2: C, Connector_PinSocket_2.54mm:PinSocket_1x02_P2.54mm_Vertical, symbol Device:C
- added C3: C_Polarized, Connector_PinSocket_2.54mm:PinSocket_1x02_P2.54mm_Vertical, symbol Device:C_Polarized
- added D1, D2, D3: LED, Connector_PinSocket_2.54mm:PinSocket_1x02_P2.54mm_Vertical, symbol Device:LED
- added J10, J11, J12, J13, J14, J15, J16, J17, J20, J23, J9: Conn_01x03_Socket, Connector_PinSocket_2.54mm:PinSocket_1x03_P2.54mm_Vertical, symbol Connector:Conn_01x03_Socket
- added J18, J19, J21: Conn_01x10_Socket, Connector_PinSocket_2.54mm:PinSocket_1x10_P2.54mm_Vertical, symbol Connector:Conn_01x10_Socket
- added J22: Conn_01x02_Socket, Connector_PinSocket_2.54mm:PinSocket_1x02_P2.54mm_Vertical, symbol Connector:Conn_01x02_Socket
- added J24: J1_B, Connector_PinSocket_2.54mm:PinSocket_1x01_P2.54mm_Vertical, symbol Connector:Conn_01x01_Pin
- added J25: J2_B, Connector_PinSocket_2.54mm:PinSocket_1x01_P2.54mm_Vertical, symbol Connector:Conn_01x01_Pin
- added J26: J3_B, Connector_PinSocket_2.54mm:PinSocket_1x01_P2.54mm_Vertical, symbol Connector:Conn_01x01_Pin
- added J27: J1_A, Connector_PinSocket_2.54mm:PinSocket_1x01_P2.54mm_Vertical, symbol Connector:Conn_01x01_Pin
- added J28: J2_A, Connector_PinSocket_2.54mm:PinSocket_1x01_P2.54mm_Vertical, symbol Connector:Conn_01x01_Pin
- added J29: J3_A, Connector_PinSocket_2.54mm:PinSocket_1x01_P2.54mm_Vertical, symbol Connector:Conn_01x01_Pin
- added J30: J4_B, Connector_PinSocket_2.54mm:PinSocket_1x01_P2.54mm_Vertical, symbol Connector:Conn_01x01_Pin
- added J31: J5_B, Connector_PinSocket_2.54mm:PinSocket_1x01_P2.54mm_Vertical, symbol Connector:Conn_01x01_Pin
- added J32: J4_A, Connector_PinSocket_2.54mm:PinSocket_1x01_P2.54mm_Vertical, symbol Connector:Conn_01x01_Pin
- added J33: J5_A, Connector_PinSocket_2.54mm:PinSocket_1x01_P2.54mm_Vertical, symbol Connector:Conn_01x01_Pin
- added J34: J6_B, Connector_PinSocket_2.54mm:PinSocket_1x01_P2.54mm_Vertical, symbol Connector:Conn_01x01_Pin
- added J35: J7_B, Connector_PinSocket_2.54mm:PinSocket_1x01_P2.54mm_Vertical, symbol Connector:Conn_01x01_Pin
- added J36: J6_A, Connector_PinSocket_2.54mm:PinSocket_1x01_P2.54mm_Vertical, symbol Connector:Conn_01x01_Pin
- added J37: J7_A, Connector_PinSocket_2.54mm:PinSocket_1x01_P2.54mm_Vertical, symbol Connector:Conn_01x01_Pin
- added J38: J9_B, Connector_PinSocket_2.54mm:PinSocket_1x01_P2.54mm_Vertical, symbol Connector:Conn_01x01_Pin
- added J39: J8_B, Connector_PinSocket_2.54mm:PinSocket_1x01_P2.54mm_Vertical, symbol Connector:Conn_01x01_Pin
- added J40: J8_A, Connector_PinSocket_2.54mm:PinSocket_1x01_P2.54mm_Vertical, symbol Connector:Conn_01x01_Pin
- added J41: J9_A, Connector_PinSocket_2.54mm:PinSocket_1x01_P2.54mm_Vertical, symbol Connector:Conn_01x01_Pin
- added J42: J10_B, Connector_PinSocket_2.54mm:PinSocket_1x01_P2.54mm_Vertical, symbol Connector:Conn_01x01_Pin
- added J43: J10_A, Connector_PinSocket_2.54mm:PinSocket_1x01_P2.54mm_Vertical, symbol Connector:Conn_01x01_Pin
- added J44: J11_B, Connector_PinSocket_2.54mm:PinSocket_1x01_P2.54mm_Vertical, symbol Connector:Conn_01x01_Pin
- added J45: J11_A, Connector_PinSocket_2.54mm:PinSocket_1x01_P2.54mm_Vertical, symbol Connector:Conn_01x01_Pin
- added J46: J12_B, Connector_PinSocket_2.54mm:PinSocket_1x01_P2.54mm_Vertical, symbol Connector:Conn_01x01_Pin
- added J47: J12_A, Connector_PinSocket_2.54mm:PinSocket_1x01_P2.54mm_Vertical, symbol Connector:Conn_01x01_Pin
- added J48: J13_B, Connector_PinSocket_2.54mm:PinSocket_1x01_P2.54mm_Vertical, symbol Connector:Conn_01x01_Pin
- added J49: J13_A, Connector_PinSocket_2.54mm:PinSocket_1x01_P2.54mm_Vertical, symbol Connector:Conn_01x01_Pin
- added J5, J6, J7, J8: Conn_01x04_Socket, Connector_PinSocket_2.54mm:PinSocket_1x04_P2.54mm_Vertical, symbol Connector:Conn_01x04_Socket
- added J50: J14_B, Connector_PinSocket_2.54mm:PinSocket_1x01_P2.54mm_Vertical, symbol Connector:Conn_01x01_Pin
- added J51: J14_A, Connector_PinSocket_2.54mm:PinSocket_1x01_P2.54mm_Vertical, symbol Connector:Conn_01x01_Pin
- added J52: J16_B, Connector_PinSocket_2.54mm:PinSocket_1x01_P2.54mm_Vertical, symbol Connector:Conn_01x01_Pin
- added J53: J15_B, Connector_PinSocket_2.54mm:PinSocket_1x01_P2.54mm_Vertical, symbol Connector:Conn_01x01_Pin
- added J54: J15_A, Connector_PinSocket_2.54mm:PinSocket_1x01_P2.54mm_Vertical, symbol Connector:Conn_01x01_Pin
- added J55: J16_A, Connector_PinSocket_2.54mm:PinSocket_1x01_P2.54mm_Vertical, symbol Connector:Conn_01x01_Pin
- added J56: J17_B, Connector_PinSocket_2.54mm:PinSocket_1x01_P2.54mm_Vertical, symbol Connector:Conn_01x01_Pin
- added J57: J17_A, Connector_PinSocket_2.54mm:PinSocket_1x01_P2.54mm_Vertical, symbol Connector:Conn_01x01_Pin
- added J58, J63: J18_A, Connector_PinSocket_2.54mm:PinSocket_1x01_P2.54mm_Vertical, symbol Connector:Conn_01x01_Pin
- added J59, J62: J19_A, Connector_PinSocket_2.54mm:PinSocket_1x01_P2.54mm_Vertical, symbol Connector:Conn_01x01_Pin
- added J60, J61: J20_A, Connector_PinSocket_2.54mm:PinSocket_1x01_P2.54mm_Vertical, symbol Connector:Conn_01x01_Pin
- added J64, J65: Conn_01x15_Socket, Connector_PinSocket_2.54mm:PinSocket_1x15_P2.54mm_Vertical, symbol Connector:Conn_01x15_Socket
- added J66: J21_A, Connector_PinSocket_2.54mm:PinSocket_1x01_P2.54mm_Vertical, symbol Connector:Conn_01x01_Pin
- added J67: J21_B, Connector_PinSocket_2.54mm:PinSocket_1x01_P2.54mm_Vertical, symbol Connector:Conn_01x01_Pin
- added J68: J22_B, Connector_PinSocket_2.54mm:PinSocket_1x01_P2.54mm_Vertical, symbol Connector:Conn_01x01_Pin
- added J69: J22_A, Connector_PinSocket_2.54mm:PinSocket_1x01_P2.54mm_Vertical, symbol Connector:Conn_01x01_Pin
- added J70: J23_B, Connector_PinSocket_2.54mm:PinSocket_1x01_P2.54mm_Vertical, symbol Connector:Conn_01x01_Pin
- added J71: J23_A, Connector_PinSocket_2.54mm:PinSocket_1x01_P2.54mm_Vertical, symbol Connector:Conn_01x01_Pin
- added R1, R2, R3: R, Connector_PinSocket_2.54mm:PinSocket_1x02_P2.54mm_Vertical, symbol Device:R
- added SW1, SW2: SW_Push, Button_Switch_THT:SW_PUSH_6mm_H5mm, symbol Switch:SW_Push
- added U1: ~, MyLibrary:STM32F446RE, symbol MyLibrary:STM32F446RE
- added U3: ~, MyLibrary:TO220F, symbol MyLibrary:NJM7800
- J1: footprint (none) -> Connector_PinSocket_2.54mm:PinSocket_1x07_P2.54mm_Vertical
- J2, J3, J4: footprint (none) -> Connector_PinSocket_2.54mm:PinSocket_1x04_P2.54mm_Vertical
Connections:
- net +3V3: now also J10.2 (Pin_2), J11.2 (Pin_2), J12.2 (Pin_2), J13.2 (Pin_2), J14.2 (Pin_2), J15.2 (Pin_2), J16.2 (Pin_2), J17.2 (Pin_2), J19.1 (Pin_1), J19.10 (Pin_10), J19.2 (Pin_2), J19.3 (Pin_3), J19.4 (Pin_4), J19.5 (Pin_5), J19.6 (Pin_6), J19.7 (Pin_7), J19.8 (Pin_8), J19.9 (Pin_9), J20.2 (Pin_2), J5.1 (Pin_1), J6.1 (Pin_1), J7.1 (Pin_1), J8.1 (Pin_1), J9.2 (Pin_2), SW1.2, SW2.2, U1.3 (3V3)
- net +5V: now also C2.1, C3.1, J69.1 (Pin_1), U1.1 (5V), U3.2 (OUT)
- net GND: now also C1.2, C2.2, C3.2, D1.1 (K), D2.1 (K), D3.1 (K), J10.3 (Pin_3), J11.3 (Pin_3), J12.3 (Pin_3), J13.3 (Pin_3), J14.3 (Pin_3), J15.3 (Pin_3), J16.3 (Pin_3), J17.3 (Pin_3), J20.3 (Pin_3), J22.1 (Pin_1), J43.1 (Pin_1), J5.2 (Pin_2), J6.2 (Pin_2), J7.2 (Pin_2), J71.1 (Pin_1), J8.2 (Pin_2), J9.3 (Pin_3), U1.2 (GND), U1.48 (GND), U1.50 (GND), U3.3 (GND)
- net RX/Serial2: now also J54.1 (Pin_1), U1.15 (RX/Serial2); no longer J1.7 (Pin_7), J2.4 (Pin_4)
- net RX/Serial3: now also J66.1 (Pin_1), U1.9 (RX/Serial3)
- net RX/Serial4: now also U1.17 (RX/Serial4)
- net SWCLK: now also J40.1 (Pin_1), U1.35 (SWCLK/PA14); no longer J1.2 (Pin_2)
- net SWDIO: now also J41.1 (Pin_1), U1.34 (SWDIO/PA13); no longer J1.4 (Pin_4)
- net TX/Serial2: now also J55.1 (Pin_1), U1.16 (TX/Serial2); no longer J1.6 (Pin_6), J2.3 (Pin_3)
- net TX/Serial3: now also J65.9 (Pin_9), U1.7 (TX/Serial3)
- net TX/Serial4: now also J57.1 (Pin_1), U1.18 (TX/Serial4); no longer J4.3 (Pin_3)
- new net: J21.2 (Pin_2), J48.1 (Pin_1)
- new net: J30.1 (Pin_1), R2.1
- new net: D2.2 (A), R2.2
- new net: J35.1 (Pin_1), J5.3 (Pin_3)
- new net: J34.1 (Pin_1), J5.4 (Pin_4)
- new net: J4.3 (Pin_3), J56.1 (Pin_1)
- new net: D1.2 (A), R1.2
- new net: J1.2 (Pin_2), J39.1 (Pin_1)
- new net: J1.4 (Pin_4), J38.1 (Pin_1)
- new net: J44.1 (Pin_1), SW1.1
- new net: J18.1 (Pin_1), J18.10 (Pin_10), J18.2 (Pin_2), J18.3 (Pin_3), J18.4 (Pin_4), J18.5 (Pin_5), J18.6 (Pin_6), J18.7 (Pin_7), J18.8 (Pin_8), J18.9 (Pin_9), J42.1 (Pin_1)
- new net: J64.2 (Pin_2), J68.1 (Pin_1)
- new net: J21.3 (Pin_3), J50.1 (Pin_1)
- new net: J64.9 (Pin_9), J67.1 (Pin_1)
- new net: J31.1 (Pin_1), R3.1
- new net: J65.13 (Pin_13), J65.14 (Pin_14), J65.15 (Pin_15), J70.1 (Pin_1)
- new net: J21.1 (Pin_1), J46.1 (Pin_1)
- new net: D3.2 (A), R3.2
- new net: J60.1 (Pin_1), J61.1 (Pin_1)
- new net: J59.1 (Pin_1), J62.1 (Pin_1)
- new net: J58.1 (Pin_1), J63.1 (Pin_1)
- new net +9V: J22.2 (Pin_2), J23.2 (Pin_2)
- new net Analog/PA4: J14.1 (Pin_1), U1.14 (Analog/PA4)
- new net Analog/PA5: J13.1 (Pin_1), U1.13 (Analog/PA5)
- new net Analog/PA6: J12.1 (Pin_1), U1.12 (Analog/PA6)
- new net Analog/PA7: J11.1 (Pin_1), U1.11 (Analog/PA7)
- new net Analog/PB1: J9.1 (Pin_1), U1.8 (Analog/PB1)
- new net Analog/PC0: J20.1 (Pin_1), U1.22 (Analog/PC0)
- new net Analog/PC1: J17.1 (Pin_1), U1.21 (Analog/PC1)
- new net Analog/PC2: J16.1 (Pin_1), U1.20 (Analog/PC2)
- new net Analog/PC3: J15.1 (Pin_1), U1.19 (Analog/PC3)
- new net Analog/PC4: J10.1 (Pin_1), U1.10 (Analog/PC4)
- new net Digital/PA11: J29.1 (Pin_1), U1.32 (Digital/PA11)
- new net Digital/PA11/sub: J21.9 (Pin_9), J26.1 (Pin_1), J32.1 (Pin_1)
- new net Digital/PA12: J21.4 (Pin_4), U1.33 (Digital/PA12)
- new net Digital/PB12: J51.1 (Pin_1), U1.6 (Digital/PB12)
- new net Digital/PB13: J49.1 (Pin_1), U1.5 (Dgital/PB13)
- new net Digital/PB14: J47.1 (Pin_1), U1.4 (Digital/PB14)
- new net Digital/PB15: J27.1 (Pin_1), U1.26 (Digital/PB15)
- new net Digital/PB15/sub: J21.7 (Pin_7), J24.1 (Pin_1), SW2.1
- new net Digital/PB5: J21.10 (Pin_10), R1.1, U1.43 (Digital/PB5)
- new net Digital/PC10: J21.5 (Pin_5), U1.37 (Digital/PC10)
- new net Digital/PC11: J21.6 (Pin_6), J45.1 (Pin_1), U1.38 (Digital/PC11)
- new net Digital/PC8: J28.1 (Pin_1), U1.29 (Digital/PC8)
- new net Digital/PC8/sub: J21.8 (Pin_8), J25.1 (Pin_1), J33.1 (Pin_1)
- new net Main9V: C1.1, J23.1 (Pin_1), U3.1 (IN)
- new net RX/Serial2/sub: J1.7 (Pin_7), J2.4 (Pin_4), J53.1 (Pin_1)
- new net RX/Serial5: J36.1 (Pin_1), U1.40 (RX/Serial5)
- new net RX/Serial6: J6.4 (Pin_4), U1.28 (RX/Serial6)
- new net SCL/I2C1: J7.4 (Pin_4), U1.46 (SCL/I2C1)
- new net SCL/I2C3: J8.4 (Pin_4), U1.31 (SCL/I2C3)
- new net SDA/I2C1: J7.3 (Pin_3), U1.47 (SDA/I2C1)
- new net SDA/I2C3: J8.3 (Pin_3), U1.30 (SDA/I2C3)
- new net TX/Serial2/sub: J1.6 (Pin_6), J2.3 (Pin_3), J52.1 (Pin_1)
- new net TX/Serial5: J37.1 (Pin_1), U1.39 (TX/Serial5)
- new net TX/Serial6: J6.3 (Pin_3), U1.27 (TX/Serial6)
- no-connect marks 8 -> 36
Other:
- moved on the sheet: J1, J2, J3, J4
